File: quickstep_controller/quickstep_controller RevI/qs_SD_Interface.sch (KiCad schematic (older format))
At the start: 17 parts, among them J201 SD_Card, U201 TS3A27518E, U202 SN74LVC1G3157DCK3

Commit message: Messing around with direct SD-MMC upload; hardware changes required and messing around with ESP3D
Other:
- note added: "NEED TO ADD POWER CONTROL TO SWITCH MODES"
Changed lines of the file:
@@
 Wire Wire Line
 	2750 3400 3400 3400
+Text Notes 6750 1550 0    100  ~ 0
+NEED TO ADD POWER CONTROL TO SWITCH MODES
 $EndSCHEMATC
