File: quickstep_controller/quickstep_controller RevII/qs_Switches.sch (KiCad schematic (older format))
At the start: 41 parts, among them Q401 NTR3C21NZT1G, Q402 NTR3C21NZT1G, U401 74HC14

Commit message: Messing around with direct SD-MMC upload; hardware changes required and messing around with ESP3D
Parts:
- renumbered C401 to C?, C402 to C?, C403 to C?, C404 to C?, C405 to C?, C408 to C?, C406 to C?, D409 to D?, D410 to D?, D406 to D?, D407 to D?, D408 to D?, D405 to D?, Q401 to Q?, Q402 to Q?, R401 to R?, R405 to R?, R402 to R?, R406 to R?, R403 to R?, R407 to R?, R404 to R?, R408 to R?, R409 to R?, R410 to R?, R411 to R?, R412 to R?, R413 to R?, R417 to R?, U401 to U?
Changed lines of the file:
@@
 EESchema Schematic File Version 4
+LIBS:quickstep_controller RevII-cache
 EELAYER 30 0
 EELAYER END
@@
 $EndDescr
 $Comp
-L Device:R R401
+L Device:R R?
 U 1 1 5E4A125F
 P 3000 1250
@@
 $EndComp
 $Comp
-L Device:R R405
+L Device:R R?
 U 1 1 5E4A1AF0
 P 3300 1550
@@
 $EndComp
 $Comp
-L Device:C C401
+L Device:C C?
 U 1 1 5E4A2A00
 P 3950 1800
@@
 Connection ~ 3000 2050
 $Comp
-L power:GND #PWR0402
+L power:GND #PWR?
 U 1 1 5E4A38DB
 P 3000 2150
@@
 	3000 1000 3000 1100
 $Comp
-L power:+3.3V #PWR0401
+L power:+3.3V #PWR?
 U 1 1 5E4A404E
 P 3000 1000
@@
 X_STOP_OUT
 $Comp
-L Device:R R402
+L Device:R R?
 U 1 1 5E4AA0CA
 P 3000 2950
@@
 $EndComp
 $Comp
-L Device:R R406
+L Device:R R?
 U 1 1 5E4AA0D0
 P 3300 3250
@@
 $EndComp
 $Comp
-L Device:C C402
+L Device:C C?
 U 1 1 5E4AA0DC
 P 3950 3500
@@
 Connection ~ 3000 3750
 $Comp
-L power:GND #PWR0404
+L power:GND #PWR?
 U 1 1 5E4AA0F5
 P 3000 3850
@@
 	3000 2700 3000 2800
 $Comp
-L power:+3.3V #PWR0403
+L power:+3.3V #PWR?
 U 1 1 5E4AA0FC
 P 3000 2700
@@
 Y_STOP_OUT
 $Comp
-L Device:R R403
+L Device:R R?
 U 1 1 5E4ACB4D
 P 3000 4650
@@
 $EndComp
 $Comp
-L Device:R R407
+L Device:R R?
 U 1 1 5E4ACB53
 P 3300 4950
@@
 $EndComp
 $Comp
-L Device:C C403
+L Device:C C?
 U 1 1 5E4ACB5F
 P 3950 5200
@@
 Connection ~ 3000 5450
 $Comp
-L power:GND #PWR0406
+L power:GND #PWR?
 U 1 1 5E4ACB78
 P 3000 5550
@@
 	3000 4400 3000 4500
 $Comp
-L power:+3.3V #PWR0405
+L power:+3.3V #PWR?
 U 1 1 5E4ACB7F
 P 3000 4400
@@
 Z_STOP_OUT
 $Comp
-L Device:R R404
+L Device:R R?
 U 1 1 5E4BA014
 P 3000 6350
@@
 $EndComp
 $Comp
-L Device:R R408
+L Device:R R?
 U 1 1 5E4BA01A
 P 3300 6650
@@
 $EndComp
 $Comp
-L Device:C C404
+L Device:C C?
 U 1 1 5E4BA026
 P 3950 6900
@@
 Connection ~ 3000 7150
 $Comp
-L power:GND #PWR0408
+L power:GND #PWR?
 U 1 1 5E4BA03F
 P 3000 7250
@@
 	3000 6100 3000 6200
 $Comp
-L power:+3.3V #PWR0407
+L power:+3.3V #PWR?
 U 1 1 5E4BA046
 P 3000 6100
@@
 FIL_SEN_OUT
 $Comp
-L 74xx:74HC14 U401
+L 74xx:74HC14 U?
 U 7 1 5E4C5ACA
 P 6850 5450
@@
 $EndComp
 $Comp
-L power:GND #PWR0411
+L power:GND #PWR?
 U 1 1 5E4F8434
 P 6850 6050
@@
 	6850 4850 6500 4850
 $Comp
-L Device:C C405
+L Device:C C?
 U 1 1 5E4FDA94
 P 6500 5100
@@
 	6500 4850 6500 4950
 $Comp
-L power:GND #PWR0409
+L power:GND #PWR?
 U 1 1 5E50010F
 P 6500 5350
@@
 Connection ~ 6850 4850
 $Comp
-L power:+3.3V #PWR0410
+L power:+3.3V #PWR?
 U 1 1 5E507496
 P 6850 4750
@@
 $EndComp
 $Comp
-L power:+3.3V #PWR0414
+L power:+3.3V #PWR?
 U 1 1 5E5086C7
 P 8200 1200
@@
 $EndComp
 $Comp
-L Custom-DiscreteSymbols:NTR3C21NZT1G Q401
+L Custom-DiscreteSymbols:NTR3C21NZT1G Q?
 U 1 1 5E518A45
 P 7300 1650
@@
 RST
 $Comp
-L power:+3.3V #PWR0415
+L power:+3.3V #PWR?
 U 1 1 5E54B6AD
 P 8200 2550
@@
 $EndComp
 $Comp
-L Device:C C408
+L Device:C C?
 U 1 1 5E54B6C5
 P 8200 1900
@@
 $EndComp
 $Comp
-L Custom-DiscreteSymbols:NTR3C21NZT1G Q402
+L Custom-DiscreteSymbols:NTR3C21NZT1G Q?
 U 1 1 5E54B6D1
 P 7300 3000
@@
 Microswitch Inputs
 $Comp
-L Device:C C406
+L Device:C C?
 U 1 1 5E56A58D
 P 6850 1650
@@
 E-stop Input (NO Switch)
 $Comp
-L Device:LED D409
+L Device:LED D?
 U 1 1 5ED61630
 P 7500 1300
@@
 $EndComp
 $Comp
-L Device:LED D410
+L Device:LED D?
 U 1 1 5ED6268E
 P 7500 2650
@@
 $EndComp
 $Comp
-L Device:LED D406
+L Device:LED D?
 U 1 1 5ED62F96
 P 4700 3450
@@
 $EndComp
 $Comp
-L Device:LED D407
+L Device:LED D?
 U 1 1 5ED64406
 P 4700 5150
@@
 $EndComp
 $Comp
-L Device:LED D408
+L Device:LED D?
 U 1 1 5ED649C2
 P 4700 6850
@@
 $EndComp
 $Comp
-L Device:LED D405
+L Device:LED D?
 U 1 1 5ED6502D
 P 4700 1750
@@
 $EndComp
 $Comp
-L Device:R R409
+L Device:R R?
 U 1 1 5ED65C85
 P 4450 2050
@@
 $EndComp
 $Comp
-L Device:R R410
+L Device:R R?
 U 1 1 5ED66AEE
 P 4450 3750
@@
 $EndComp
 $Comp
-L Device:R R411
+L Device:R R?
 U 1 1 5ED67203
 P 4450 5450
@@
 $EndComp
 $Comp
-L Device:R R412
+L Device:R R?
 U 1 1 5ED67724
 P 4450 7150
@@
 $EndComp
 $Comp
-L Device:R R413
+L Device:R R?
 U 1 1 5ED67C90
 P 7950 1300
@@
 $EndComp
 $Comp
-L Device:R R417
+L Device:R R?
 U 1 1 5ED711EA
 P 7950 2650
@@
 Connection ~ 3950 2050
 $Comp
-L power:PWR_FLAG #FLG0401
+L power:PWR_FLAG #FLG?
 U 1 1 5EB24DA1
 P 6850 4850
@@
 $EndComp
 $Comp
-L 74xx:74HC14 U401
+L 74xx:74HC14 U?
 U 1 1 5F07FDD2
 P 4350 3250
@@
 $EndComp
 $Comp
-L 74xx:74HC14 U401
+L 74xx:74HC14 U?
 U 4 1 5F081C1E
 P 4350 6650
@@
 $EndComp
 $Comp
-L 74xx:74HC14 U401
+L 74xx:74HC14 U?
 U 5 1 5F083494
 P 4350 1550
@@
 $EndComp
 $Comp
-L 74xx:74HC14 U401
+L 74xx:74HC14 U?
 U 6 1 5F084F37
 P 4350 4950
